File: Kicad/FullAdder_8Bit/FullAdder_8Bit.kicad_pcb (KiCad board)
At the start: 2 copper layers, 83 x 97 mm, 366 parts, among them J5 Conn_01x29_Pin, Q10 NPN, Q100 NPN, Q101 NPN, Q102 NPN, Q103 NPN, Q104 NPN, Q105 NPN, Q106 NPN, Q107 NPN, Q108 NPN, Q109 NPN, Q11 NPN, Q110 NPN, Q111 NPN, Q112 NPN, Q113 NPN, Q114 NPN, Q115 NPN, Q116 NPN, Q117 NPN, Q118 NPN, Q119 NPN, Q12 NPN, Q120 NPN, Q121 NPN, Q122 NPN, Q123 NPN, Q124 NPN, Q125 NPN, Q126 NPN, Q127 NPN, Q128 NPN, Q129 NPN, Q13 NPN, Q130 NPN, Q131 NPN, Q132 NPN, Q133 NPN, Q134 NPN, Q135 NPN, Q136 NPN, Q137 NPN, Q138 NPN, Q139 NPN, Q14 NPN, Q140 NPN, Q141 NPN, Q142 NPN, Q143 NPN, Q144 NPN, Q145 NPN, Q146 NPN, Q147 NPN, Q148 NPN, Q15 NPN, Q16 NPN, Q17 NPN, Q18 NPN, Q19 NPN, Q20 NPN, Q21 NPN, Q22 NPN, Q23 NPN, Q24 NPN, Q25 NPN, Q26 NPN, Q27 NPN, Q28 NPN, Q29 NPN, Q3 NPN, Q30 NPN, Q31 NPN, Q32 NPN, Q33 NPN, Q34 NPN, Q35 NPN, Q36 NPN, Q37 NPN, Q38 NPN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

Commit message: Did some routing!
Parts:
- removed J5: Conn_01x29_Pin, Connector_PinHeader_2.54mm:PinHeader_1x29_P2.54mm_Horizontal
- added J1: Conn_01x30_Pin, Connector_PinHeader_2.54mm:PinHeader_1x30_P2.54mm_Horizontal, F.Cu at (141.0, 109.3)
Connections:
- net Carry3 renamed AuxiliaryCarry
Routing:
- net UseCarryFlag: track 0.00 -> 40.9 mm
- net CarryIn_AdderBit0: track 0.00 -> 38.8 mm, vias 0 -> 6
- net Carry6: track 0.00 -> 33.7 mm, vias 0 -> 3
- net Net-(Q118-C): track 0.00 -> 32.6 mm, vias 0 -> 1
- net Net-(Q3-C): track 0.00 -> 31.5 mm, vias 0 -> 3
- net Net-(Q21-C): track 0.00 -> 31.0 mm, vias 0 -> 4
- net Carry4: track 0.00 -> 27.3 mm, vias 0 -> 1
- net Net-(Q31-C): track 0.00 -> 26.8 mm, vias 0 -> 2
- net Net-(Q76-C): track 0.00 -> 26.5 mm, vias 0 -> 2
- net Net-(Q11-C): track 0.00 -> 25.1 mm, vias 0 -> 2
- net Net-(Q78-C): track 0.00 -> 24.8 mm
- net Net-(Q115-C): track 0.00 -> 22.4 mm
- net Net-(Q117-C): track 0.00 -> 19.9 mm, vias 0 -> 1
- net Net-(Q45-C): track 0.00 -> 18.7 mm, vias 0 -> 2
- net Net-(Q127-C): track 0.00 -> 18.7 mm
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- added copper zone on B.Cu, net +5V
- added copper zone on F.Cu, net GND
Other:
- board size 83 x 97 mm -> 83 x 97.5 mm

Commit message: Finished the ADD PCB
Parts:
- J1: moved to B.Cu
- moved J1 73.3 mm to (141.2, 36.1)
- moved R190 0.34 mm to (209.1, 79.0)
- moved R170 0.31 mm to (203.6, 89.4)
- moved R144 0.30 mm to (191.4, 39.6)
- moved R123 0.30 mm to (187.0, 104.0)
- moved R107 0.28 mm to (173.0, 96.8)
- moved R102 0.27 mm to (167.3, 103.4)
- moved R142 0.27 mm to (192.3, 65.8)
- moved R148 0.25 mm to (197.0, 33.6)
- moved R50 0.25 mm to (170.7, 55.6)
- moved R54 0.25 mm to (170.7, 62.6)
- moved R126 0.23 mm to (192.3, 72.8)
- moved R208 0.23 mm to (214.0, 33.0)
- moved R217 0.23 mm to (214.6, 47.0)
- moved R94 0.21 mm to (161.7, 96.4)
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Connections:
- Q148 pad 1: Net-(Q148-C) -> CarryIn_AdderBit0
- R222 pad 1: Net-(Q148-C) -> CarryIn_AdderBit0
- R222 pad 2: CarryIn_AdderBit0 -> Carry Flag
Routing:
- net +5V: track 6.06 -> 282.4 mm, vias 2 -> 69
- net Out_Bit4: track 5.12 -> 208.4 mm, vias 0 -> 1
- net AuxiliaryCarry: track 5.02 -> 195.3 mm, vias 0 -> 14
- net Out_Bit5: track 5.04 -> 180.7 mm, vias 0 -> 1
- net Out_Bit0: track 5.05 -> 162.1 mm, vias 0 -> 4
- net Out_Bit6: track 5.04 -> 149.8 mm, vias 0 -> 1
- net Out_Bit1: track 5.08 -> 136.7 mm, vias 0 -> 3
- net B_Bit6: track 0.00 -> 123.2 mm, vias 0 -> 8
- net Out_Bit7: track 5.50 -> 122.3 mm, vias 0 -> 1
- net B_Bit7: track 0.00 -> 101.3 mm, vias 0 -> 6
- net Out_Bit2: track 5.09 -> 105.3 mm, vias 0 -> 3
- net A_Bit4: track 9.42 -> 91.7 mm, vias 0 -> 4
- net Carry7: track 5.30 -> 81.3 mm, vias 0 -> 6
- net A_Bit7: track 9.19 -> 79.8 mm, vias 2 -> 12
- net Out_Bit3: track 5.17 -> 75.7 mm, vias 0 -> 3
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Other:
- board size 83 x 97.5 mm -> 90 x 99.9 mm
- board text added: "5V"
- board text added: "ADD Module"
- board text added: "Auxilary Carry"
- board text added: "Carry Flag"
- board text added: "CarryOut"
- board text added: "GND"
- board text added: "Use Carry Flag"
- board text added: "| A0-7 |"
- board text added: "| B0-7 |"
- board text added: "|OUT0-7|"
