File: Kicad/FullAdder_8Bit/FullAdder_8Bit.kicad_sch (KiCad schematic)
At the start: 366 parts, among them J5 Conn_01x29_Pin, Q10 NPN, Q100 NPN, Q101 NPN, Q102 NPN, Q103 NPN, Q104 NPN, Q105 NPN, Q106 NPN, Q107 NPN, Q108 NPN, Q109 NPN, Q11 NPN, Q110 NPN, Q111 NPN, Q112 NPN, Q113 NPN, Q114 NPN, Q115 NPN, Q116 NPN, Q117 NPN, Q118 NPN, Q119 NPN, Q12 NPN, Q120 NPN, Q121 NPN, Q122 NPN, Q123 NPN, Q124 NPN, Q125 NPN, Q126 NPN, Q127 NPN, Q128 NPN, Q129 NPN, Q13 NPN, Q130 NPN, Q131 NPN, Q132 NPN, Q133 NPN, Q134 NPN, Q135 NPN, Q136 NPN, Q137 NPN, Q138 NPN, Q139 NPN, Q14 NPN, Q140 NPN, Q141 NPN, Q142 NPN, Q143 NPN, Q144 NPN, Q145 NPN, Q146 NPN, Q147 NPN, Q148 NPN, Q15 NPN, Q16 NPN, Q17 NPN, Q18 NPN, Q19 NPN, Q20 NPN, Q21 NPN, Q22 NPN, Q23 NPN, Q24 NPN, Q25 NPN, Q26 NPN, Q27 NPN, Q28 NPN, Q29 NPN, Q3 NPN, Q30 NPN, Q31 NPN, Q32 NPN, Q33 NPN, Q34 NPN, Q35 NPN, Q36 NPN, Q37 NPN, Q38 NPN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

Commit message: Did some routing!
Parts:
- removed J5: Conn_01x29_Pin, Connector_PinHeader_2.54mm:PinHeader_1x29_P2.54mm_Horizontal, symbol Connector:Conn_01x29_Pin
- added J1: Conn_01x30_Pin, Connector_PinHeader_2.54mm:PinHeader_1x30_P2.54mm_Horizontal, symbol Connector:Conn_01x30_Pin
Connections:
- net +5V: now also J1.17 (Pin_17)
- net A_Bit0: now also J1.1 (Pin_1)
- net A_Bit1: now also J1.2 (Pin_2)
- net A_Bit2: now also J1.3 (Pin_3)
- net A_Bit3: now also J1.4 (Pin_4)
- net A_Bit4: now also J1.5 (Pin_5)
- net A_Bit5: now also J1.6 (Pin_6)
- net A_Bit6: now also J1.7 (Pin_7)
- net A_Bit7: now also J1.8 (Pin_8)
- net B_Bit0: now also J1.9 (Pin_9)
- net B_Bit1: now also J1.10 (Pin_10)
- net B_Bit2: now also J1.11 (Pin_11)
- net B_Bit3: now also J1.12 (Pin_12)
- net B_Bit4: now also J1.13 (Pin_13)
- net B_Bit5: now also J1.14 (Pin_14)
- net B_Bit6: now also J1.15 (Pin_15)
- net B_Bit7: now also J1.16 (Pin_16)
- net Carry Flag: now also J1.19 (Pin_19)
- net Carry7: now also J1.29 (Pin_29)
- net GND: now also J1.18 (Pin_18)
- net Out_Bit0: now also J1.21 (Pin_21)
- net Out_Bit1: now also J1.22 (Pin_22)
- net Out_Bit2: now also J1.23 (Pin_23)
- net Out_Bit3: now also J1.24 (Pin_24)
- net Out_Bit4: now also J1.25 (Pin_25)
- net Out_Bit5: now also J1.26 (Pin_26)
- net Out_Bit6: now also J1.27 (Pin_27)
- net Out_Bit7: now also J1.28 (Pin_28)
- net UseCarryFlag: now also J1.20 (Pin_20)
- net Carry3 renamed AuxiliaryCarry
- net AuxiliaryCarry: now also J1.30 (Pin_30)
Changed lines of the file:
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@@
 	)
 	(junction
+		(at 311.15 215.9)
+		(diameter 0)
+		(color 0 0 0 0)
+	)
+	(junction
 		(at 146.05 207.01)
 		(diameter 0)
@@
 	(wire
 		(pts
+			(xy 311.15 215.9) (xy 312.42 215.9)
+		)
+		(stroke
+			(width 0)
+			(type default)
+		)
+	)
+	(wire
+		(pts
 			(xy 293.37 106.68) (xy 293.37 104.14)
 		)
@@
 	(wire
 		(pts
-			(xy 311.15 212.09) (xy 311.15 228.6)
+			(xy 311.15 212.09) (xy 311.15 215.9)
 		)
 		(stroke
@@
 	(wire
 		(pts
+			(xy 311.15 215.9) (xy 311.15 228.6)
+		)
+		(stroke
+			(width 0)
+			(type default)
+		)
+	)
+	(wire
+		(pts
 			(xy 187.96 213.36) (xy 196.85 213.36)
 		)
@@
 	(rectangle
 		(start 73.025 194.31)
-		(end 323.215 251.46)
+		(end 329.565 251.46)
 		(stroke
 			(width 0)
@@
 		)
 	)
+	(global_label "AuxiliaryCarry"
+		(shape input)
+		(at 25.4 120.65 0)
+		(fields_autoplaced yes)
+		(effects
+			(font
+				(size 1.27 1.27)
+			)
+			(justify left)
+		)
+		(property "Intersheetrefs" "${INTERSHEET_REFS}"
+			(at 41.3875 120.65 0)
+			(effects
+				(font
+					(size 1.27 1.27)
+				)
+				(justify left)
+				(hide yes)
+			)
+		)
+	)
 	(global_label "Out_Bit4"
 		(shape input)
@@
 		)
 	)
+	(global_label "AuxiliaryCarry"
+		(shape input)
+		(at 312.42 215.9 0)
+		(fields_autoplaced yes)
+		(effects
+			(font
+				(size 1.27 1.27)
+			)
+			(justify left)
+		)
+		(property "Intersheetrefs" "${INTERSHEET_REFS}"
+			(at 328.4075 215.9 0)
+			(effects
+				(font
+					(size 1.27 1.27)
+				)
+				(justify left)
+				(hide yes)
+			)
+		)
+	)
 	(global_label "A_Bit4"
 		(shape input)
@@
 	)
 	(symbol
-		(lib_id "Connector:Conn_01x29_Pin")
-		(at 20.32 82.55 0)
-		(unit 1)
-		(exclude_from_sim no)
-		(in_bom yes)
-		(on_board yes)
-		(dnp no)
-		(fields_autoplaced yes)
-		(property "Reference" "J5"
-			(at 20.955 41.91 0)
-			(effects
-				(font
-					(size 1.27 1.27)
-				)
-			)
-		)
-		(property "Value" "Conn_01x29_Pin"
-			(at 20.955 44.45 0)
-			(effects
-				(font
-					(size 1.27 1.27)
-				)
-			)
-		)
-		(property "Footprint" "Connector_PinHeader_2.54mm:PinHeader_1x29_P2.54mm_Horizontal"
-			(at 20.32 82.55 0)
-			(effects
-				(font
-					(size 1.27 1.27)
-				)
-				(hide yes)
-			)
-		)
-		(property "Datasheet" "~"
-			(at 20.32 82.55 0)
-			(effects
-				(font
-					(size 1.27 1.27)
-				)
-				(hide yes)
-			)
-		)
-		(property "Description" "Generic connector, single row, 01x29, script generated"
-			(at 20.32 82.55 0)
-			(effects
-				(font
-					(size 1.27 1.27)
-				)
-				(hide yes)
-			)
-		)
-		(pin "6"
-		)
-		(pin "10"
-		)
-		(pin "29"
-		)
-		(pin "14"
-		)
-		(pin "16"
-		)
-		(pin "4"
-		)
-		(pin "3"
-		)
-		(pin "24"
-		)
-		(pin "26"
-		)
-		(pin "19"
-		)
-		(pin "21"
-		)
-		(pin "25"
-		)
-		(pin "1"
-		)
-		(pin "12"
-		)
-		(pin "13"
-		)
-		(pin "22"
-		)
-		(pin "9"
-		)
-		(pin "20"
-		)
-		(pin "8"
-		)
-		(pin "28"
-		)
-		(pin "5"
-		)
-		(pin "7"
-		)
-		(pin "17"
-		)
-		(pin "27"
-		)
-		(pin "2"
-		)
-		(pin "23"
-		)
-		(pin "18"
-		)
-		(pin "11"
-		)
-		(pin "15"
-		)
-		(instances
-			(project ""
-				(path "/d162130f-3a1c-4d14-8b0f-52f8ec57a6b4"
-					(reference "J5")
-					(unit 1)
-				)
-			)
-		)
-	)
-	(symbol
 		(lib_id "Simulation_SPICE:NPN")
 		(at 515.62 265.43 0)
@@
 					(unit 1)
 				)
+			)
+		)
+	)
+	(symbol
+		(lib_id "Connector:Conn_01x30_Pin")
+		(at 20.32 82.55 0)
+		(unit 1)
+		(exclude_from_sim no)
+		(in_bom yes)
+		(on_board yes)
+		(dnp no)
+		(fields_autoplaced yes)
+		(property "Reference" "J1"
+			(at 20.955 41.91 0)
+			(effects
+				(font
+					(size 1.27 1.27)
+				)
+			)
+		)
+		(property "Value" "Conn_01x30_Pin"
+			(at 20.955 44.45 0)
+			(effects
+				(font
+					(size 1.27 1.27)
+				)
+			)
+		)
+		(property "Footprint" "Connector_PinHeader_2.54mm:PinHeader_1x30_P2.54mm_Horizontal"
+			(at 20.32 82.55 0)
+			(effects
+				(font
+					(size 1.27 1.27)
+				)
+				(hide yes)
+			)
+		)
+		(property "Datasheet" "~"
+			(at 20.32 82.55 0)
+			(effects
+				(font
+					(size 1.27 1.27)
+				)
+				(hide yes)
+			)
+		)
+		(property "Description" "Generic connector, single row, 01x30, script generated"
+			(at 20.32 82.55 0)
+			(effects
+				(font
+					(size 1.27 1.27)
+				)
+				(hide yes)
+			)
+		)
+		(pin "19"
+		)
+		(pin "20"
+		)
+		(pin "11"
+		)
+		(pin "1"
+		)
+		(pin "10"
+		)
+		(pin "12"
+		)
+		(pin "13"
+		)
+		(pin "14"
+		)
+		(pin "15"
+		)
+		(pin "16"
+		)
+		(pin "18"
+		)
+		(pin "17"
+		)
+		(pin "2"
+		)
+		(pin "21"
+		)
+		(pin "22"
+		)
+		(pin "23"
+		)
+		(pin "24"
+		)
+		(pin "25"
+		)
+		(pin "26"
+		)
+		(pin "27"
+		)
+		(pin "28"
+		)
+		(pin "29"
+		)
+		(pin "3"
+		)
+		(pin "30"
+		)
+		(pin "4"
+		)
+		(pin "5"
+		)
+		(pin "6"
+		)
+		(pin "9"
+		)
+		(pin "7"
+		)
+		(pin "8"
+		)
+		(instances
+			(project ""
+				(path "/d162130f-3a1c-4d14-8b0f-52f8ec57a6b4"
+					(reference "J1")
+					(unit 1)
+				)

Commit message: Finished the ADD PCB
Connections:
- net Carry Flag: now also R222.2
- net CarryIn_AdderBit0: now also Q148.1 (C), R222.1; no longer R222.2

Commit message: Made a backup; removed all traces and put parts where they need to be. starting routing again
Parts:
- removed J1: Conn_01x30_Pin, Connector_PinHeader_2.54mm:PinHeader_1x30_P2.54mm_Horizontal, symbol Connector:Conn_01x30_Pin
- added J2: Conn_01x31_Pin, Connector_PinHeader_2.54mm:PinHeader_1x31_P2.54mm_Horizontal, symbol Connector:Conn_01x31_Pin
- added Q1, Q149, Q150, Q151, Q152, Q153, Q154, Q155, Q156, Q157, Q158, Q159, Q160, Q161, Q162, Q163, Q164, Q165, Q166, Q167, Q168, Q169, Q170, Q171, Q172, Q173, Q174, Q175, Q176, Q177, Q178, Q179, Q180, Q181, Q182, Q183, Q184, Q185, Q186, Q187, Q188, Q189, Q190, Q191, Q192, Q193, Q194, Q195, Q196, Q197, Q198, Q199, Q2, Q200, Q201, Q202, Q203, Q204, Q205, Q206, Q207, Q208, Q209, Q210, Q211, Q212, Q213, Q214, Q215, Q216, Q217, Q218, Q219, Q220, Q221, Q222, Q223, Q224, Q225, Q226, Q227: NPN, Package_TO_SOT_THT:TO-92, symbol Simulation_SPICE:NPN
- added R1, R2, R223, R224, R225, R226, R227, R228, R229, R230, R231, R232, R233, R234, R235, R236, R237, R238, R239, R240, R241, R242, R243, R244, R245, R246, R247, R248, R249, R250, R251, R252, R253, R254, R255, R256, R257, R258, R259, R260, R261, R262, R263, R264, R265, R266, R267, R268, R269, R270, R271, R272, R273, R274, R275, R276, R277, R278, R279, R280, R281, R282, R283, R284, R285, R286, R287, R288, R289, R290, R291, R292, R293, R294, R295, R296, R297, R298, R299, R3, R300, R301, R302, R303, R304, R305, R306, R307, R308, R309, R310, R311, R312, R313, R314, R315, R316, R317, R318, R319, R320, R321, R322, R323, R324, R325, R326, R327, R328, R329, R330, R331, R332, R333, R334, R335, R336, R337, R338, R339, R340, R341, R342, R343, R344, R345: 1kΩ, Resistor_SMD:R_0603_1608Metric, symbol Device:R
Connections:
- net +5V: now also J2.17 (Pin_17), R2.1, R224.1, R227.1, R230.1, R232.2, R235.1, R239.1, R240.1, R244.1, R247.2, R250.1, R251.1, R258.1, R259.1, R260.1, R261.1, R268.1, R269.1, R274.2, R275.2, R280.1, R281.1, R282.1, R283.1, R296.1, R297.1, R298.1, R299.1, R300.1, R301.1, R302.1, R303.1, R316.1, R317.1, R318.1, R319.1, R328.2, R329.2, R330.2, R331.2, R333.1, R337.1, R338.1, R342.1, R345.2
- net A_Bit0: now also J2.1 (Pin_1)
- net A_Bit1: now also J2.2 (Pin_2)
- net A_Bit2: now also J2.3 (Pin_3)
- net A_Bit3: now also J2.4 (Pin_4)
- net A_Bit4: now also J2.5 (Pin_5)
- net A_Bit5: now also J2.6 (Pin_6)
- net A_Bit6: now also J2.7 (Pin_7)
- net A_Bit7: now also J2.8 (Pin_8)
- net AuxiliaryCarry: now also J2.31 (Pin_31)
- net B_Bit0: now also Q155.1 (C), R232.1
- net B_Bit1: now also Q164.1 (C), R247.1
- net B_Bit2: now also Q181.1 (C), R274.1
- net B_Bit3: now also Q182.1 (C), R275.1
- net B_Bit4: now also Q215.1 (C), R328.1
- net B_Bit5: now also Q216.1 (C), R329.1
- net B_Bit6: now also Q217.1 (C), R330.1
- net B_Bit7: now also Q218.1 (C), R331.1
- net Carry7: now also J2.30 (Pin_30)
- net GND: now also J2.18 (Pin_18), Q1.3 (E), Q149.3 (E), Q150.3 (E), Q151.3 (E), Q152.3 (E), Q153.3 (E), Q154.3 (E), Q155.3 (E), Q156.3 (E), Q157.3 (E), Q158.3 (E), Q159.3 (E), Q160.3 (E), Q161.3 (E), Q162.3 (E), Q163.3 (E), Q164.3 (E), Q165.3 (E), Q166.3 (E), Q167.3 (E), Q168.3 (E), Q169.3 (E), Q170.3 (E), Q171.3 (E), Q172.3 (E), Q173.3 (E), Q174.3 (E), Q175.3 (E), Q176.3 (E), Q177.3 (E), Q178.3 (E), Q179.3 (E), Q180.3 (E), Q181.3 (E), Q182.3 (E), Q183.3 (E), Q184.3 (E), Q185.3 (E), Q186.3 (E), Q187.3 (E), Q188.3 (E), Q189.3 (E), Q190.3 (E), Q191.3 (E), Q192.3 (E), Q193.3 (E), Q194.3 (E), Q195.3 (E), Q196.3 (E), Q197.3 (E), Q198.3 (E), Q199.3 (E), Q2.3 (E), Q200.3 (E), Q201.3 (E), Q202.3 (E), Q203.3 (E), Q204.3 (E), Q205.3 (E), Q206.3 (E), Q207.3 (E), Q208.3 (E), Q209.3 (E), Q210.3 (E), Q211.3 (E), Q212.3 (E), Q213.3 (E), Q214.3 (E), Q215.3 (E), Q216.3 (E), Q217.3 (E), Q218.3 (E), Q219.3 (E), Q220.3 (E), Q221.3 (E), Q222.3 (E), Q223.3 (E), Q224.3 (E), Q225.3 (E), Q226.3 (E), Q227.3 (E)
- net Out_Bit0: now also J2.22 (Pin_22)
- net Out_Bit1: now also J2.23 (Pin_23)
- net Out_Bit2: now also J2.24 (Pin_24)
- net Out_Bit3: now also J2.25 (Pin_25)
- net Out_Bit4: now also J2.26 (Pin_26)
- net Out_Bit5: now also J2.27 (Pin_27)
- net Out_Bit6: now also J2.28 (Pin_28)
- net Out_Bit7: now also J2.29 (Pin_29)
- net UseCarryFlag: now also J2.20 (Pin_20)
- net Carry Flag renamed CarryFlag
- net CarryFlag: now also Q227.1 (C), R345.1
- new net: Q198.1 (C), Q206.1 (C), R303.2, R323.1
- new net: Q2.2 (B), R1.2
- new net: Q186.1 (C), Q190.1 (C), R283.2, R294.1, R295.1
- new net: Q186.2 (B), R279.2
- new net: Q215.2 (B), R324.1
- new net: Q178.1 (C), Q180.1 (C), R269.2, R273.2
- new net: Q180.2 (B), R271.2
- new net: Q193.1 (C), Q201.1 (C), R298.2, R313.1
- new net: Q201.2 (B), R306.2
- new net: Q165.1 (C), Q167.1 (C), R250.2, R254.1, R255.1
- new net: Q167.2 (B), R252.2
- new net: Q184.1 (C), Q188.1 (C), R281.2, R290.1, R291.1
- new net: Q194.1 (C), Q202.1 (C), R299.2, R321.1
- new net: Q194.2 (B), R291.2
- new net: Q208.1 (C), Q212.1 (C), R317.2, R325.2
- new net: Q212.2 (B), R321.2
- new net: Q210.1 (C), Q214.1 (C), R319.2, R327.2
- new net: Q214.2 (B), R323.2
- new net: Q153.1 (C), Q154.1 (C), R230.2, R233.2
- new net: Q219.1 (C), Q220.1 (C), R333.2, R335.1, R336.1
- new net: Q227.2 (B), R344.1
- new net: Q225.1 (C), Q226.1 (C), R342.2, R344.2
- new net: Q207.1 (C), Q211.1 (C), R316.2, R324.2
- new net: Q218.2 (B), R327.1
- new net: Q149.1 (C), Q2.1 (C), R2.2, R223.1, R226.1
- new net: Q151.2 (B), R226.2
- new net: Q196.1 (C), Q204.1 (C), R301.2, R322.1
- new net: Q196.2 (B), R293.2
- new net: Q197.1 (C), Q205.1 (C), R302.2, R315.1
- new net: Q205.2 (B), R310.2
- new net: Q166.1 (C), Q168.1 (C), R251.2, R256.1, R257.1
- new net: Q150.2 (B), R225.2
- new net: Q216.2 (B), R325.1
- new net: Q182.2 (B), R273.1
- new net: Q151.1 (C), Q152.1 (C), R227.2, R231.1
- new net: Q152.2 (B), R228.2
- new net: Q159.1 (C), Q161.1 (C), R240.2, R245.1
- new net: Q161.2 (B), R242.2
- new net: Q217.2 (B), R326.1
- new net: Q154.2 (B), R231.2
- new net: Q183.1 (C), Q187.1 (C), R280.2, R288.1, R289.1
- new net: Q191.2 (B), R288.2
- new net: Q185.2 (B), R278.2
- new net: Q207.2 (B), R312.2
- new net: Q224.2 (B), R340.2
- new net: Q155.2 (B), R233.1
- new net: Q199.2 (B), R304.2
- new net: Q164.2 (B), R246.1
- new net: Q162.1 (C), Q163.1 (C), R244.2, R246.2
- new net: Q156.1 (C), Q157.1 (C), R235.2, R237.1, R238.1
- new net: Q197.2 (B), R294.2
- new net: Q225.2 (B), R341.2
- new net: Q170.1 (C), Q174.1 (C), R259.2, R270.1
- new net: Q174.2 (B), R263.2
- new net: Q175.2 (B), R264.2
- new net: Q204.2 (B), R309.2
- new net: Q222.1 (C), Q224.1 (C), R338.2, R343.1
- new net: Q226.2 (B), R343.2
- new net: Q171.2 (B), R256.2
- new net: Q185.1 (C), Q189.1 (C), R282.2, R292.1, R293.1
- new net: Q169.1 (C), Q173.1 (C), R258.2, R266.1
- new net: Q177.2 (B), R266.2
- new net: Q149.2 (B), R3.2
- new net: Q1.1 (C), Q150.1 (C), R224.2, R229.1
- new net: Q153.2 (B), R229.2
- new net: Q220.2 (B), R334.2
- new net: Q172.1 (C), Q176.1 (C), R261.2, R271.1
- new net: Q210.2 (B), R315.2
- new net: Q209.1 (C), Q213.1 (C), R318.2, R326.2
- new net: Q208.2 (B), R313.2
- new net: Q173.2 (B), R262.2
- new net: Q222.2 (B), R336.2
- new net: Q221.1 (C), Q223.1 (C), R337.2, R341.1
- new net: Q223.2 (B), R339.2
- new net: Q163.2 (B), R245.2
- new net: Q219.2 (B), R332.2
- new net: Q189.2 (B), R286.2
- new net: Q184.2 (B), R277.2
- new net: Q172.2 (B), R257.2
- new net: Q192.1 (C), Q200.1 (C), R297.2, R320.1
- new net: Q213.2 (B), R322.2
- new net: Q168.2 (B), R253.2
- new net: Q158.1 (C), Q160.1 (C), R239.2, R243.1
- new net: Q160.2 (B), R241.2
- new net: Q178.2 (B), R267.2
- new net: Q177.1 (C), Q179.1 (C), R268.2, R272.2
- new net: Q179.2 (B), R270.2
- new net: Q156.2 (B), R234.2
- new net: Q1.2 (B), R223.2
- new net: Q206.2 (B), R311.2
- new net: Q171.1 (C), Q175.1 (C), R260.2, R267.1
- new net: Q195.1 (C), Q203.1 (C), R300.2, R314.1
- new net: Q195.2 (B), R292.2
- new net: Q165.2 (B), R248.2
- new net: Q202.2 (B), R307.2
- new net: Q203.2 (B), R308.2
- new net: Q190.2 (B), R287.2
- new net: Q188.2 (B), R285.2
- new net: Q158.2 (B), R237.2
- new net: Q200.2 (B), R305.2
- new net: Q157.2 (B), R236.2
- new net: Q221.2 (B), R335.2
- new net: Q176.2 (B), R265.2
- new net: Q191.1 (C), Q199.1 (C), R296.2, R312.1
- new net: Q183.2 (B), R276.2
- new net: Q181.2 (B), R272.1
- new net: Q192.2 (B), R289.2
- new net: Q193.2 (B), R290.2
- new net: Q162.2 (B), R243.2
- new net: Q159.2 (B), R238.2
- new net: Q169.2 (B), R254.2
- new net: Q187.2 (B), R284.2
- new net: Q170.2 (B), R255.2
- new net: Q211.2 (B), R320.2
- new net: Q209.2 (B), R314.2
- new net: Q198.2 (B), R295.2
- new net: Q166.2 (B), R249.2
- new net B_Bit0In: J2.9 (Pin_9), R1.1, R225.1
- new net B_Bit1In: J2.10 (Pin_10), R234.1, R241.1
- new net B_Bit2In: J2.11 (Pin_11), R248.1, R262.1
- new net B_Bit3In: J2.12 (Pin_12), R249.1, R264.1
- new net B_Bit4In: J2.13 (Pin_13), R276.1, R304.1
- new net B_Bit5In: J2.14 (Pin_14), R277.1, R306.1
- new net B_Bit6In: J2.15 (Pin_15), R278.1, R308.1
- new net B_Bit7In: J2.16 (Pin_16), R279.1, R310.1
- new net CarryFlagIn: J2.19 (Pin_19), R332.1, R339.1
- new net IsSub: J2.21 (Pin_21), R228.1, R236.1, R242.1, R252.1, R253.1, R263.1, R265.1, R284.1, R285.1, R286.1, R287.1, R3.1, R305.1, R307.1, R309.1, R311.1, R334.1, R340.1
Other:
- note added: "8 Bit Adder"
- note added: "Bit 0 XOR IsSub = Bit 0 to use"
- note added: "Bit 1 XOR IsSub = Bit 1 to use"
- note added: "Bit 2 XOR IsSub = Bit 2 to use"
- note added: "Bit 3 XOR IsSub = Bit 3 to use"
- note added: "Bit 4 XOR IsSub = Bit 4 to use"
- note added: "Bit 5 XOR IsSub = Bit 5 to use"
- note added: "Bit 6 XOR IsSub = Bit 6 to use"
- note added: "Bit 7 XOR IsSub = Bit 7 to use"
- note added: "XOR selection for subtraction"
- moved on the sheet: Q10, Q100, Q101, Q102, Q103, Q104, Q105, Q106, Q107, Q108, Q109, Q11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

Commit message: Revert "Made a backup; removed all traces and put parts where they need to be. starting routing again"
This reverts commit 2ef9f42e64e6a7f49d503f8bd060bf19175d52bc.
Parts:
- removed J2: Conn_01x31_Pin, Connector_PinHeader_2.54mm:PinHeader_1x31_P2.54mm_Horizontal, symbol Connector:Conn_01x31_Pin
- removed Q1, Q149, Q150, Q151, Q152, Q153, Q154, Q155, Q156, Q157, Q158, Q159, Q160, Q161, Q162, Q163, Q164, Q165, Q166, Q167, Q168, Q169, Q170, Q171, Q172, Q173, Q174, Q175, Q176, Q177, Q178, Q179, Q180, Q181, Q182, Q183, Q184, Q185, Q186, Q187, Q188, Q189, Q190, Q191, Q192, Q193, Q194, Q195, Q196, Q197, Q198, Q199, Q2, Q200, Q201, Q202, Q203, Q204, Q205, Q206, Q207, Q208, Q209, Q210, Q211, Q212, Q213, Q214, Q215, Q216, Q217, Q218, Q219, Q220, Q221, Q222, Q223, Q224, Q225, Q226, Q227: NPN, Package_TO_SOT_THT:TO-92, symbol Simulation_SPICE:NPN
- removed R1, R2, R223, R224, R225, R226, R227, R228, R229, R230, R231, R232, R233, R234, R235, R236, R237, R238, R239, R240, R241, R242, R243, R244, R245, R246, R247, R248, R249, R250, R251, R252, R253, R254, R255, R256, R257, R258, R259, R260, R261, R262, R263, R264, R265, R266, R267, R268, R269, R270, R271, R272, R273, R274, R275, R276, R277, R278, R279, R280, R281, R282, R283, R284, R285, R286, R287, R288, R289, R290, R291, R292, R293, R294, R295, R296, R297, R298, R299, R3, R300, R301, R302, R303, R304, R305, R306, R307, R308, R309, R310, R311, R312, R313, R314, R315, R316, R317, R318, R319, R320, R321, R322, R323, R324, R325, R326, R327, R328, R329, R330, R331, R332, R333, R334, R335, R336, R337, R338, R339, R340, R341, R342, R343, R344, R345: 1kΩ, Resistor_SMD:R_0603_1608Metric, symbol Device:R
- added J1: Conn_01x30_Pin, Connector_PinHeader_2.54mm:PinHeader_1x30_P2.54mm_Horizontal, symbol Connector:Conn_01x30_Pin
Connections:
- net +5V: now also J1.17 (Pin_17)
- net A_Bit0: now also J1.1 (Pin_1)
- net A_Bit1: now also J1.2 (Pin_2)
- net A_Bit2: now also J1.3 (Pin_3)
- net A_Bit3: now also J1.4 (Pin_4)
- net A_Bit4: now also J1.5 (Pin_5)
- net A_Bit5: now also J1.6 (Pin_6)
- net A_Bit6: now also J1.7 (Pin_7)
- net A_Bit7: now also J1.8 (Pin_8)
- net AuxiliaryCarry: now also J1.30 (Pin_30)
- net B_Bit0: now also J1.9 (Pin_9)
- net B_Bit1: now also J1.10 (Pin_10)
- net B_Bit2: now also J1.11 (Pin_11)
- net B_Bit3: now also J1.12 (Pin_12)
- net B_Bit4: now also J1.13 (Pin_13)
- net B_Bit5: now also J1.14 (Pin_14)
- net B_Bit6: now also J1.15 (Pin_15)
- net B_Bit7: now also J1.16 (Pin_16)
- net Carry7: now also J1.29 (Pin_29)
- net GND: now also J1.18 (Pin_18)
- net Out_Bit0: now also J1.21 (Pin_21)
- net Out_Bit1: now also J1.22 (Pin_22)
- net Out_Bit2: now also J1.23 (Pin_23)
- net Out_Bit3: now also J1.24 (Pin_24)
- net Out_Bit4: now also J1.25 (Pin_25)
- net Out_Bit5: now also J1.26 (Pin_26)
- net Out_Bit6: now also J1.27 (Pin_27)
- net Out_Bit7: now also J1.28 (Pin_28)
- net UseCarryFlag: now also J1.20 (Pin_20)
- net CarryFlag renamed Carry Flag
- net Carry Flag: now also J1.19 (Pin_19)
Other:
- note removed: "8 Bit Adder"
- note removed: "Bit 0 XOR IsSub = Bit 0 to use"
- note removed: "Bit 1 XOR IsSub = Bit 1 to use"
- note removed: "Bit 2 XOR IsSub = Bit 2 to use"
- note removed: "Bit 3 XOR IsSub = Bit 3 to use"
- note removed: "Bit 4 XOR IsSub = Bit 4 to use"
- note removed: "Bit 5 XOR IsSub = Bit 5 to use"
- note removed: "Bit 6 XOR IsSub = Bit 6 to use"
- note removed: "Bit 7 XOR IsSub = Bit 7 to use"
- note removed: "XOR selection for subtraction"
- moved on the sheet: Q10, Q100, Q101, Q102, Q103, Q104, Q105, Q106, Q107, Q108, Q109, Q11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
