File: Kicad/FullSubtractor_8Bit/FullSubtractor_8Bit.kicad_pcb (KiCad board)
At the start: 2 copper layers, 90 x 99.9 mm, 393 parts, among them J1 Conn_01x30_Pin, Q1 NPN, Q10 NPN, Q100 NPN, Q101 NPN, Q102 NPN, Q103 NPN, Q104 NPN, Q105 NPN, Q106 NPN, Q107 NPN, Q108 NPN, Q109 NPN, Q11 NPN, Q110 NPN, Q111 NPN, Q112 NPN, Q113 NPN, Q114 NPN, Q115 NPN, Q116 NPN, Q117 NPN, Q118 NPN, Q119 NPN, Q12 NPN, Q120 NPN, Q121 NPN, Q122 NPN, Q123 NPN, Q124 NPN, Q125 NPN, Q126 NPN, Q127 NPN, Q128 NPN, Q129 NPN, Q13 NPN, Q130 NPN, Q131 NPN, Q132 NPN, Q133 NPN, Q134 NPN, Q135 NPN, Q136 NPN, Q137 NPN, Q138 NPN, Q139 NPN, Q14 NPN, Q140 NPN, Q141 NPN, Q142 NPN, Q143 NPN, Q144 NPN, Q145 NPN, Q146 NPN, Q149 NPN, Q15 NPN, Q150 NPN, Q151 NPN, Q152 NPN, Q153 NPN, Q154 NPN, Q155 NPN, Q156 NPN, Q157 NPN, Q16 NPN, Q17 NPN, Q18 NPN, Q19 NPN, Q2 NPN, Q20 NPN, Q21 NPN, Q22 NPN, Q23 NPN, Q24 NPN, Q25 NPN, Q26 NPN, Q27 NPN, Q28 NPN, Q29 NPN, Q3 NPN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

Commit message: 8 Bit Subtractor Done!
Parts:
- moved Q1 150.4 mm to (218.0, 109.1)
- moved R1 150.4 mm to (216.9, 107.4)
- moved R2 150.4 mm to (219.6, 110.5)
- moved R237 103.3 mm to (200.7, 111.6)
- moved Q155 103.3 mm to (199.1, 110.0)
- moved R233 103.3 mm to (198.0, 108.2)
- moved R230 0.76 mm to (197.0, 36.8)
- moved Q151 0.73 mm to (150.3, 107.8)
- moved R227 0.73 mm to (149.3, 106.2)
- moved R229 0.73 mm to (151.9, 109.5)
Routing:
- net B_Bit6In: track 0.00 -> 118.0 mm, vias 0 -> 6
- net B_Bit7In: track 0.00 -> 111.4 mm, vias 0 -> 4
- net B_Bit6: track 125.2 -> 20.8 mm, vias 8 -> 2
- net BorrowOut: track 0.00 -> 91.3 mm, vias 0 -> 6
- net B_Bit7: track 101.3 -> 19.7 mm, vias 6 -> 2
- net (no net): track 81.3 -> 0.00 mm, vias 6 -> 0
- net +5V: track 303.4 -> 370.4 mm, vias 73 -> 85
- net Borrow7: track 0.00 -> 17.9 mm, vias 0 -> 2
- net Net-(Q155-B): track 0.00 -> 1.73 mm
- net Net-(Q1-B): track 0.00 -> 1.70 mm
- net Net-(Q118-C): track 32.6 -> 33.6 mm
- net Net-(Q11-C): track 24.9 -> 25.7 mm
- net Net-(Q117-C): track 29.4 -> 30.2 mm
- net Net-(Q31-C): track 27.1 -> 27.7 mm
- net B_Bit4In: track 80.1 -> 80.6 mm, vias 7 -> 6
Other:
- board text added: "SUB Module"
- board text removed: "ADD Module"
